File: pcb/U3A_rs422.kicad_sch (KiCad schematic)
At the start: 17 parts, among them J1 Conn_02x05_Odd_Even, J2 Conn_01x07_Socket, J4 Conn_01x08_Socket, U2 THVD1452DR, U3 THVD1452DR

Commit message: Change vendor of parts
Parts:
- H1, H2: Vendor HTL, DigiKey -> HTL; VendorId 100991, 100993, 732-12987-ND -> 100991, 100993, 103622
- U2, U3: VendorId 296-THVD1452DRCT-ND -> 103640
Changed lines of the file:
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@@
       (effects (font (size 1.27 1.27)) hide)
     )
-    (property "Vendor" "HTL, DigiKey" (at 215.9 151.13 0)
-      (effects (font (size 1.27 1.27)) hide)
-    )
-    (property "VendorId" "100991, 100993, 732-12987-ND" (at 215.9 151.13 0)
+    (property "Vendor" "HTL" (at 215.9 151.13 0)
+      (effects (font (size 1.27 1.27)) hide)
+    )
+    (property "VendorId" "100991, 100993, 103622" (at 215.9 151.13 0)
       (effects (font (size 1.27 1.27)) hide)
     )
@@
       (effects (font (size 1.27 1.27)) hide)
     )
-    (property "Vendor" "HTL, DigiKey" (at 205.74 151.13 0)
-      (effects (font (size 1.27 1.27)) hide)
-    )
-    (property "VendorId" "100991, 100993, 732-12987-ND" (at 205.74 151.13 0)
+    (property "Vendor" "HTL" (at 205.74 151.13 0)
+      (effects (font (size 1.27 1.27)) hide)
+    )
+    (property "VendorId" "100991, 100993, 103622" (at 205.74 151.13 0)
       (effects (font (size 1.27 1.27)) hide)
     )
@@
       (effects (font (size 1.27 1.27)) hide)
     )
-    (property "VendorId" "296-THVD1452DRCT-ND" (at 116.84 107.95 0)
+    (property "VendorId" "103640" (at 116.84 107.95 0)
       (effects (font (size 1.27 1.27)) hide)
     )
@@
       (effects (font (size 1.27 1.27)) hide)
     )
-    (property "VendorId" "296-THVD1452DRCT-ND" (at 116.84 57.15 0)
-      (effects (font (size 1.27 1.27)) hide)
-    )
+    (property "VendorId" "103640" (at 116.84 57.15 0)
+      (effects (font (size 1.27 1.27)) hide)
+    )

Commit message: Update to KiCAD 9
Parts:
- FID1, FID2, FID3, FID4, H1, H2: now left out of the parts list

Commit message: Rename/Add/Remove bom fields
Parts:
- C1: HTL (none) -> 100140; Vendor HTL -> (none); VendorId 100140 -> (none)
- C2, C3: HTL (none) -> 100128; Vendor HTL -> (none); VendorId 100128 -> (none)
- H1, H2: HTL (none) -> 100991, 100993, 103622; Vendor HTL -> (none); VendorId 100991, 100993, 103622 -> (none)
- J1: HTL (none) -> 101532; Vendor HTL -> (none); VendorId 101532 -> (none)
- J2, J4: HTL (none) -> 101546; Vendor HTL -> (none); VendorId 101546 -> (none)
- R1: HTL (none) -> 102967; Vendor HTL -> (none); VendorId 102967 -> (none)
- R2, R3: HTL (none) -> 102933; Vendor HTL -> (none); VendorId 102933 -> (none)
- U2, U3: HTL (none) -> 103640; Vendor DigiKey -> (none); VendorId 103640 -> (none)
Changed lines of the file:
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@@
 			)
 		)
-		(property "Vendor" "HTL"
-			(at 127 177.8 0)
-			(effects
-				(font
-					(size 1.27 1.27)
-				)
-				(hide yes)
-			)
-		)
-		(property "VendorId" "100128"
+		(property "HTL" "100128"
 			(at 127 177.8 0)
 			(effects
@@
 			)
 		)
-		(property "Vendor" "HTL"
-			(at 215.9 151.13 0)
-			(effects
-				(font
-					(size 1.27 1.27)
-				)
-				(hide yes)
-			)
-		)
-		(property "VendorId" "100991, 100993, 103622"
-			(at 215.9 151.13 0)
+		(property "HTL" "100991, 100993, 103622"
+			(at 215.9 151.13 90)
 			(effects
 				(font
@@
 			)
 		)
-		(property "Vendor" "HTL"
-			(at 143.51 50.8 0)
-			(effects
-				(font
-					(size 1.27 1.27)
-				)
-				(hide yes)
-			)
-		)
-		(property "VendorId" "102933"
-			(at 143.51 50.8 0)
+		(property "HTL" "102933"
+			(at 143.51 50.8 90)
 			(effects
 				(font
@@
 			)
 		)
-		(property "Vendor" "HTL"
-			(at 83.82 120.65 0)
-			(effects
-				(font
-					(size 1.27 1.27)
-				)
-				(hide yes)
-			)
-		)
-		(property "VendorId" "102967"
-			(at 83.82 120.65 0)
+		(property "HTL" "102967"
+			(at 83.82 120.65 90)
 			(effects
 				(font
@@
 			)
 		)
-		(property "Vendor" ""
-			(at 254 152.4 0)
-			(effects
-				(font
-					(size 1.27 1.27)
-				)
-				(hide yes)
-			)
-		)
-		(property "VendorId" ""
-			(at 254 152.4 0)
-			(effects
-				(font
-					(size 1.27 1.27)
-				)
-				(hide yes)
-			)
-		)
 		(instances
 			(project "U3A_rs422"
@@
 			)
 		)
-		(property "Vendor" ""
-			(at 228.6 152.4 0)
-			(effects
-				(font
-					(size 1.27 1.27)
-				)
-				(hide yes)
-			)
-		)
-		(property "VendorId" ""
-			(at 228.6 152.4 0)
-			(effects
-				(font
-					(size 1.27 1.27)
-				)
-				(hide yes)
-			)
-		)
 		(instances
 			(project "U3A_rs422"
@@
 					(size 1.27 1.27)
 				)
-			)
-		)
-		(property "Vendor" ""
-			(at 266.7 152.4 0)
-			(effects
-				(font
-					(size 1.27 1.27)
-				)
-				(hide yes)
-			)
-		)
-		(property "VendorId" ""
-			(at 266.7 152.4 0)
-			(effects
-				(font
-					(size 1.27 1.27)
-				)
-				(hide yes)
 			)
 		)
@@
 			)
 		)
-		(property "Vendor" "HTL"
-			(at 101.6 177.8 0)
-			(effects
-				(font
-					(size 1.27 1.27)
-				)
-				(hide yes)
-			)
-		)
-		(property "VendorId" "100140"
+		(property "HTL" "100140"
 			(at 101.6 177.8 0)
 			(effects
@@
 					(size 1.27 1.27)
 				)
-			)
-		)
-		(property "Vendor" ""
-			(at 241.3 152.4 0)
-			(effects
-				(font
-					(size 1.27 1.27)
-				)
-				(hide yes)
-			)
-		)
-		(property "VendorId" ""
-			(at 241.3 152.4 0)
-			(effects
-				(font
-					(size 1.27 1.27)
-				)
-				(hide yes)
 			)
 		)
@@
 			)
 		)
-		(property "Vendor" "HTL"
-			(at 205.74 151.13 0)
-			(effects
-				(font
-					(size 1.27 1.27)
-				)
-				(hide yes)
-			)
-		)
-		(property "VendorId" "100991, 100993, 103622"
-			(at 205.74 151.13 0)
+		(property "HTL" "100991, 100993, 103622"
+			(at 205.74 151.13 90)
 			(effects
 				(font
@@
 			)
 		)
-		(property "Vendor" "DigiKey"
-			(at 116.84 107.95 0)
-			(effects
-				(font
-					(size 1.27 1.27)
-				)
-				(hide yes)
-			)
-		)
-		(property "VendorId" "103640"
+		(property "HTL" "103640"
 			(at 116.84 107.95 0)
 			(effects
@@
 			)
 		)
-		(property "Vendor" "HTL"
-			(at 170.18 82.55 0)
-			(effects
-				(font
-					(size 1.27 1.27)
-				)
-				(hide yes)
-			)
-		)
-		(property "VendorId" "101532"
+		(property "HTL" "101532"
 			(at 170.18 82.55 0)
 			(effects
@@
 			)
 		)
-		(property "Vendor" "HTL"
-			(at 114.3 177.8 0)
-			(effects
-				(font
-					(size 1.27 1.27)
-				)
-				(hide yes)
-			)
-		)
-		(property "VendorId" "100128"
+		(property "HTL" "100128"
 			(at 114.3 177.8 0)
 			(effects
@@
 			)
 		)
-		(property "Vendor" "HTL"
-			(at 93.98 154.94 0)
-			(effects
-				(font
-					(size 1.27 1.27)
-				)
-				(hide yes)
-			)
-		)
-		(property "VendorId" "101546"
-			(at 93.98 154.94 0)
+		(property "HTL" "101546"
+			(at 93.98 154.94 90)
 			(effects
 				(font
@@
 			)
 		)
-		(property "Vendor" "DigiKey"
-			(at 116.84 57.15 0)
-			(effects
-				(font
-					(size 1.27 1.27)
-				)
-				(hide yes)
-			)
-		)
-		(property "VendorId" "103640"
+		(property "HTL" "103640"
 			(at 116.84 57.15 0)
 			(effects
@@
 			)
 		)
-		(property "Vendor" "HTL"
-			(at 69.85 86.36 0)
-			(effects
-				(font
-					(size 1.27 1.27)
-				)
-				(hide yes)
-			)
-		)
-		(property "VendorId" "101546"
-			(at 69.85 86.36 0)
+		(property "HTL" "101546"
+			(at 69.85 86.36 90)
 			(effects
 				(font
@@
 			)
 		)
-		(property "Vendor" "HTL"
-			(at 143.51 101.6 0)
-			(effects
-				(font
-					(size 1.27 1.27)
-				)
-				(hide yes)
-			)
-		)
-		(property "VendorId" "102933"
-			(at 143.51 101.6 0)
-			(effects
-				(font
+		(property "HTL" "102933"
+			(at 143.51 101.6 90)
+			(effects
+				(font
